File: PCB/SensorLights/SensorLights.sch (KiCad schematic (older format))
At the start: 34 parts, among them J1 Signal Power, J2 Board Power, J3 Green Signal, J4 Red Signal, J5 Manual Stop, Q1 RFP50N06LE, Q2 RFP50N06LE, SW1 Address, U1 HC-SR04, U2 ESP32_DevKit_V4

Commit message: added potentiometers for setting of the sensor distance
Other:
- note added: "Span"
- note added: "Start"
Changed lines of the file:
@@
 Wire Wire Line
 	3800 5300 4000 5300
+Text Notes 2200 7100 0    50   ~ 0
+Start
+Text Notes 2900 7100 0    50   ~ 0
+Span
 $EndSCHEMATC
